File: Nvidia_Jetson_Nano-Framos_FSM_IMX296-Adapter.kicad_pcb (KiCad board)
At the start: 2 copper layers, 27.6 x 27.4 mm, 34 parts, among them J1 DF40HC(4.0)-60DS-0.4V(51), J1 DF40HC_4.0_-60DS-0.4V_51_, J2 1-1734248-5, J3 CLK_SEL, J4 EXTENSION, SW1 MASTER_SLAVE, U1 LP5907MFX-1.8, U1 LP5907QMFX-3.8Q1, U2 LP5907MFX-1.2, U3 SN74LVC1G14DBV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

Commit message: Update schematic and layout
Connections:
- net /SCL renamed /CAM_SCL
- net /SDA renamed /CAM_SDA
- J1 pad 21: /I2C_SCL__I2C_0_SCL -> /SCL_1V8
- J1 pad 27: /I2C_SDA__I2C_0_SDA -> /SDA_1V8
- J1 pad 39: /MCLK0_INCK -> /INCK
- J3 pad 2: /MCLK0_INCK -> /INCK
