File: Nvidia_Jetson_Nano-Framos_FSM_IMX296-Adapter.sch (KiCad schematic (older format))
At the start: 27 parts, among them J1 DF40HC_4.0_-60DS-0.4V_51_, J2 1-1734248-5, J3 CLK_SEL, J4 EXTENSION, SW1 MASTER_SLAVE, U1 LP5907MFX-1.8, U2 LP5907MFX-1.2, U3 SN74LVC1G14DBV, U4 DMG1024UV-7, X1 TXC-7C

Commit message: Update schematic and layout
Connections:
- net labels added: CAM_SCL, CAM_SDA, INCK
- net labels removed: I2C_SCL__I2C_0_SCL, I2C_SDA__I2C_0_SDA, MCLK0_INCK, SCL, SDA
- wire segments 178 -> 177
- no-connect marks 32 -> 33
Other:
- moved on the sheet: R9, U4
Changed lines of the file:
@@
 Text Label 3550 2050 0    50   ~ 0
 TOUT1
-Text Label 1350 2150 0    50   ~ 0
-I2C_SCL__I2C_0_SCL
+Text Label 1900 2150 0    50   ~ 0
+SCL_1V8
 Text Label 1900 2250 0    50   ~ 0
 XCE
@@
 Text Label 3550 2350 0    50   ~ 0
 TOUT2
-Text Label 1350 2450 0    50   ~ 0
-I2C_SDA__I2C_0_SDA
+Text Label 1900 2450 0    50   ~ 0
+SDA_1V8
 Text Label 3550 2650 0    50   ~ 0
 TOUT0
@@
 Wire Wire Line
 	1300 3750 2650 3750
-Wire Wire Line
-	1300 2150 2650 2150
-Wire Wire Line
-	1300 2450 2650 2450
 NoConn ~ 4350 1950
 NoConn ~ 1850 2250
@@
 $EndComp
 Text Label 1900 3050 0    50   ~ 0
-MCLK0_INCK
+INCK
 Wire Wire Line
 	2650 3050 1850 3050
@@
 	-1   0    0    1
 $EndComp
-Wire Wire Line
-	3250 5750 3800 5750
 Text Label 3300 5750 0    50   ~ 0
-MCLK0_INCK
+INCK
 Wire Wire Line
 	3300 5650 3250 5650
@@
 MIPI_CSI_CLK0_N__D_CLK_0_P
 Text Label 6650 2950 0    50   ~ 0
-SCL
+CAM_SCL
 Text Label 6650 3050 0    50   ~ 0
-SDA
+CAM_SDA
 $Comp
 L power:GND #PWR0101
@@
 L power:+1V8 #PWR0106
 U 1 1 5FCE1BFB
-P 10550 2400
-F 0 "#PWR0106" H 10550 2250 50  0001 C CNN
-F 1 "+1V8" H 10565 2573 50  0000 C CNN
-F 2 "" H 10550 2400 50  0001 C CNN
-F 3 "" H 10550 2400 50  0001 C CNN
-	1    10550 2400
-	1    0    0    -1
-$EndComp
-Wire Wire Line
-	8700 2700 8900 2700
-Wire Wire Line
-	9900 3000 10300 3000
-Text Label 9900 3000 0    50   ~ 0
+P 10800 2400
+F 0 "#PWR0106" H 10800 2250 50  0001 C CNN
+F 1 "+1V8" H 10815 2573 50  0000 C CNN
+F 2 "" H 10800 2400 50  0001 C CNN
+F 3 "" H 10800 2400 50  0001 C CNN
+	1    10800 2400
+	1    0    0    -1
+$EndComp
+Text Label 10150 3000 0    50   ~ 0
 SCL_1V8
 Text Label 8550 2400 0    50   ~ 0
 SDA_1V8
 Wire Wire Line
-	8500 3000 8900 3000
-Wire Wire Line
-	9900 2400 10300 2400
+	10150 2400 10550 2400
 Text Label 8550 3000 0    50   ~ 0
-SCL
-Text Label 9900 2400 0    50   ~ 0
-SDA
+CAM_SCL
+Text Label 10150 2400 0    50   ~ 0
+CAM_SDA
 NoConn ~ 3550 1150
 NoConn ~ 3550 1250
@@
 L DMG1024UV-7:DMG1024UV-7 U4
 U 1 1 5FAD1AAD
-P 9400 2700
-F 0 "U4" H 9400 3267 50  0000 C CNN
-F 1 "DMG1024UV-7" H 9400 3176 50  0000 C CNN
-F 2 "footprints:DMG1024UV-7" H 9400 2700 50  0001 L BNN
-F 3 "" H 9400 2700 50  0001 L BNN
-F 4 "IPC-7351B" H 9400 2700 50  0001 L BNN "STANDARD"
-F 5 "Diodes Incorporated" H 9400 2700 50  0001 L BNN "MANUFACTURER"
-F 6 "5-2" H 9400 2700 50  0001 L BNN "PARTREV"
-	1    9400 2700
+P 9650 2700
+F 0 "U4" H 9650 3267 50  0000 C CNN
+F 1 "DMG1024UV-7" H 9650 3176 50  0000 C CNN
+F 2 "footprints:DMG1024UV-7" H 9650 2700 50  0001 L BNN
+F 3 "" H 9650 2700 50  0001 L BNN
+F 4 "IPC-7351B" H 9650 2700 50  0001 L BNN "STANDARD"
+F 5 "Diodes Incorporated" H 9650 2700 50  0001 L BNN "MANUFACTURER"
+F 6 "5-2" H 9650 2700 50  0001 L BNN "PARTREV"
+	1    9650 2700
 	1    0    0    -1
 $EndComp
@@
 	8250 2800 8500 2800
 Wire Wire Line
-	8500 2400 8900 2400
-Wire Wire Line
 	8500 2400 8500 2450
 Wire Wire Line
@@
 L Device:R_US R9
 U 1 1 5FBB6C3D
-P 10300 2800
-F 0 "R9" V 10095 2800 50  0000 C CNN
-F 1 "2k2" V 10186 2800 50  0000 C CNN
-F 2 "Resistor_SMD:R_0603_1608Metric" V 10340 2790 50  0001 C CNN
-F 3 "~" H 10300 2800 50  0001 C CNN
-	1    10300 2800
-	1    0    0    -1
-$EndComp
-Wire Wire Line
-	10300 2600 10300 2650
-Wire Wire Line
-	10300 2950 10300 3000
-Wire Wire Line
-	10100 2700 10100 2600
-Wire Wire Line
-	10100 2600 10300 2600
-Wire Wire Line
-	9900 2700 10100 2700
-Wire Wire Line
-	10550 2400 10550 2600
-Wire Wire Line
-	10550 2600 10300 2600
-Connection ~ 10300 2600
+P 10800 2800
+F 0 "R9" V 10595 2800 50  0000 C CNN
+F 1 "2k2" V 10686 2800 50  0000 C CNN
+F 2 "Resistor_SMD:R_0603_1608Metric" V 10840 2790 50  0001 C CNN
+F 3 "~" H 10800 2800 50  0001 C CNN
+	1    10800 2800
+	1    0    0    -1
+$EndComp
+Wire Wire Line
+	10350 2700 10350 2600
+Wire Wire Line
+	10150 2700 10350 2700
 Wire Wire Line
 	7650 5400 7850 5400
@@
 Connection ~ 8550 5250
 $Comp
-L power:+1V8 #PWR?
+L power:+1V8 #PWR0109
 U 1 1 5FDC0C4A
 P 1150 1450
-F 0 "#PWR?" H 1150 1300 50  0001 C CNN
+F 0 "#PWR0109" H 1150 1300 50  0001 C CNN
 F 1 "+1V8" H 1165 1623 50  0000 C CNN
 F 2 "" H 1150 1450 50  0001 C CNN
@@
 	1850 1850 2650 1850
 NoConn ~ 2650 1950
+NoConn ~ 8650 1500
+Wire Wire Line
+	8500 2400 9150 2400
+Wire Wire Line
+	8700 2700 9150 2700
+Wire Wire Line
+	8500 3000 9150 3000
+Wire Wire Line
+	10800 3000 10800 2950
+Wire Wire Line
+	10350 2600 10800 2600
+Wire Wire Line
+	10800 2400 10800 2600
+Connection ~ 10800 2600
+Wire Wire Line
+	10800 2600 10800 2650
+Wire Wire Line
+	10150 3000 10800 3000
+Wire Wire Line
+	2650 2150 1850 2150
+Wire Wire Line
+	2650 2450 1850 2450
+Wire Wire Line
+	3250 5750 3500 5750
 $EndSCHEMATC
